File: Solar Panel/SolarCellX_v2/SolarCellX_v2.sch (EAGLE design)
At the start: 17 parts

Commit message: SolarCell X first complete revision
Parts:
- removed D6: SB_DIODE, Solar:SB_DIODE
- removed U$10, U$11: BURNER, Burner:BURNER
- removed U$9: B5B-EH-A(LF)(SN), Solar:B5B-EH-A(LF)(SN)
- added 1: SLMD121H04L, Solar:SLMD121H04L
- added U$1: 6PIN_MOLEX, Solar:6PIN_MOLEX
Connections:
- removed net V_BURN: U$10.IN, U$9.P$3
- new net N$1: U$1.P$2, U$1.P$3
- net GND: now also U$1.P$1; no longer 21.P$1, 22.P$1, D3.POS, U$11.IN, U$9.P$4
- net N$3: now also 21.P$1, 22.P$1, D3.POS; no longer D5.POS
- net N$4: now also 1.P$1; no longer D6.POS
- net N$6: now also 1.P$2, D5.POS; no longer U$9.P$1, U$9.P$5
- net V_SOLAR: now also U$1.P$5; no longer D6.NEG, U$9.P$2
Changed lines of the file:
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@@
 <part name="D4" library="Solar" deviceset="SB_DIODE" device=""/>
 <part name="D5" library="Solar" deviceset="SB_DIODE" device=""/>
-<part name="D6" library="Solar" deviceset="SB_DIODE" device=""/>
-<part name="U$9" library="Solar" deviceset="B5B-EH-A(LF)(SN)" device=""/>
-<part name="U$10" library="Burner" deviceset="BURNER" device=""/>
-<part name="U$11" library="Burner" deviceset="BURNER" device=""/>
+<part name="U$1" library="Solar" deviceset="6PIN_MOLEX" device=""/>
+<part name="1" library="Solar" deviceset="SLMD121H04L" device=""/>
 </parts>
 <sheets>
@@
 <attribute name="VALUE" x="30.48" y="63.5" size="1.778" layer="95" rot="R90"/>
 </instance>
-<instance part="D6" gate="G$1" x="60.96" y="66.04" smashed="yes" rot="R90">
-<attribute name="NAME" x="59.055" y="63.754" size="1.778" layer="95" rot="R90"/>
-<attribute name="VALUE" x="66.04" y="63.5" size="1.778" layer="95" rot="R90"/>
-</instance>
-<instance part="U$9" gate="G$1" x="116.84" y="38.1" smashed="yes"/>
-<instance part="U$10" gate="G$1" x="91.44" y="38.1" smashed="yes" rot="R180"/>
-<instance part="U$11" gate="G$1" x="101.6" y="38.1" smashed="yes"/>
+<instance part="U$1" gate="G$1" x="114.3" y="40.64" smashed="yes"/>
+<instance part="1" gate="G$1" x="63.5" y="58.42" smashed="yes" rot="R90"/>
 </instances>
 <busses>
@@
 <net name="GND" class="0">
 <segment>
-<pinref part="U$9" gate="G$1" pin="P$4"/>
 <wire x1="111.76" y1="43.18" x2="109.22" y2="43.18" width="0.1524" layer="91"/>
-<wire x1="109.22" y1="43.18" x2="109.22" y2="20.32" width="0.1524" layer="91"/>
-<wire x1="109.22" y1="20.32" x2="109.22" y2="10.16" width="0.1524" layer="91"/>
-<wire x1="109.22" y1="10.16" x2="60.96" y2="10.16" width="0.1524" layer="91"/>
-<wire x1="60.96" y1="10.16" x2="25.4" y2="10.16" width="0.1524" layer="91"/>
-<wire x1="25.4" y1="10.16" x2="25.4" y2="22.86" width="0.1524" layer="91"/>
+<wire x1="109.22" y1="43.18" x2="109.22" y2="10.16" width="0.1524" layer="91"/>
+<wire x1="109.22" y1="10.16" x2="25.4" y2="10.16" width="0.1524" layer="91"/>
+<label x="114.3" y="25.4" size="1.778" layer="95"/>
 <pinref part="11" gate="G$1" pin="P$1"/>
-<wire x1="25.4" y1="22.86" x2="15.24" y2="22.86" width="0.1524" layer="91"/>
+<pinref part="D1" gate="G$1" pin="POS"/>
 <pinref part="12" gate="G$1" pin="P$1"/>
 <wire x1="25.4" y1="22.86" x2="35.56" y2="22.86" width="0.1524" layer="91"/>
 <junction x="25.4" y="22.86"/>
-<pinref part="D1" gate="G$1" pin="POS"/>
 <wire x1="25.4" y1="22.86" x2="25.4" y2="27.94" width="0.1524" layer="91"/>
-<pinref part="D3" gate="G$1" pin="POS"/>
-<wire x1="60.96" y1="25.4" x2="60.96" y2="22.86" width="0.1524" layer="91"/>
-<junction x="60.96" y="10.16"/>
-<pinref part="21" gate="G$1" pin="P$1"/>
-<wire x1="60.96" y1="22.86" x2="60.96" y2="10.16" width="0.1524" layer="91"/>
-<wire x1="60.96" y1="22.86" x2="50.8" y2="22.86" width="0.1524" layer="91"/>
-<junction x="60.96" y="22.86"/>
-<pinref part="22" gate="G$1" pin="P$1"/>
-<wire x1="60.96" y1="22.86" x2="71.12" y2="22.86" width="0.1524" layer="91"/>
-<label x="114.3" y="25.4" size="1.778" layer="95"/>
-<pinref part="U$11" gate="G$1" pin="IN"/>
-<wire x1="101.6" y1="33.02" x2="101.6" y2="20.32" width="0.1524" layer="91"/>
-<wire x1="101.6" y1="20.32" x2="109.22" y2="20.32" width="0.1524" layer="91"/>
-<junction x="109.22" y="20.32"/>
+<wire x1="25.4" y1="22.86" x2="15.24" y2="22.86" width="0.1524" layer="91"/>
+<wire x1="25.4" y1="10.16" x2="25.4" y2="22.86" width="0.1524" layer="91"/>
+<pinref part="U$1" gate="G$1" pin="P$1"/>
 </segment>
 </net>
@@
 <segment>
 <pinref part="D2" gate="G$1" pin="NEG"/>
-<pinref part="D5" gate="G$1" pin="POS"/>
 <wire x1="25.4" y1="50.8" x2="25.4" y2="53.34" width="0.1524" layer="91"/>
 <pinref part="13" gate="G$1" pin="P$2"/>
-<wire x1="25.4" y1="53.34" x2="25.4" y2="63.5" width="0.1524" layer="91"/>
 <wire x1="25.4" y1="53.34" x2="15.24" y2="53.34" width="0.1524" layer="91"/>
 <junction x="25.4" y="53.34"/>
 <pinref part="14" gate="G$1" pin="P$2"/>
 <wire x1="25.4" y1="53.34" x2="35.56" y2="53.34" width="0.1524" layer="91"/>
+<wire x1="25.4" y1="53.34" x2="25.4" y2="58.42" width="0.1524" layer="91"/>
+<wire x1="25.4" y1="58.42" x2="43.18" y2="58.42" width="0.1524" layer="91"/>
+<wire x1="43.18" y1="58.42" x2="43.18" y2="15.24" width="0.1524" layer="91"/>
+<pinref part="21" gate="G$1" pin="P$1"/>
+<pinref part="22" gate="G$1" pin="P$1"/>
+<pinref part="D3" gate="G$1" pin="POS"/>
+<wire x1="60.96" y1="25.4" x2="60.96" y2="22.86" width="0.1524" layer="91"/>
+<junction x="60.96" y="22.86"/>
+<wire x1="60.96" y1="22.86" x2="71.12" y2="22.86" width="0.1524" layer="91"/>
+<wire x1="60.96" y1="22.86" x2="50.8" y2="22.86" width="0.1524" layer="91"/>
+<wire x1="43.18" y1="15.24" x2="60.96" y2="15.24" width="0.1524" layer="91"/>
+<wire x1="60.96" y1="15.24" x2="60.96" y2="22.86" width="0.1524" layer="91"/>
 </segment>
 </net>
@@
 <wire x1="60.96" y1="53.34" x2="71.12" y2="53.34" width="0.1524" layer="91"/>
 <junction x="60.96" y="53.34"/>
-<pinref part="D6" gate="G$1" pin="POS"/>
-<wire x1="60.96" y1="53.34" x2="60.96" y2="63.5" width="0.1524" layer="91"/>
+<pinref part="1" gate="G$1" pin="P$1"/>
+<wire x1="60.96" y1="55.88" x2="60.96" y2="53.34" width="0.1524" layer="91"/>
 </segment>
 </net>
@@
 <net name="V_SOLAR" class="0">
 <segment>
-<pinref part="D6" gate="G$1" pin="NEG"/>
-<wire x1="60.96" y1="68.58" x2="60.96" y2="78.74" width="0.1524" layer="91"/>
-<wire x1="60.96" y1="78.74" x2="83.82" y2="78.74" width="0.1524" layer="91"/>
 <pinref part="D5" gate="G$1" pin="NEG"/>
 <wire x1="25.4" y1="68.58" x2="25.4" y2="78.74" width="0.1524" layer="91"/>
-<wire x1="25.4" y1="78.74" x2="60.96" y2="78.74" width="0.1524" layer="91"/>
-<junction x="60.96" y="78.74"/>
+<wire x1="25.4" y1="78.74" x2="83.82" y2="78.74" width="0.1524" layer="91"/>
 <wire x1="83.82" y1="78.74" x2="83.82" y2="53.34" width="0.1524" layer="91"/>
-<pinref part="U$9" gate="G$1" pin="P$2"/>
 <wire x1="83.82" y1="53.34" x2="111.76" y2="53.34" width="0.1524" layer="91"/>
 <label x="88.9" y="53.34" size="1.778" layer="95"/>
+<pinref part="U$1" gate="G$1" pin="P$5"/>
 </segment>
 </net>
-<net name="V_BURN" class="0">
+<net name="N$1" class="0">
 <segment>
-<pinref part="U$9" gate="G$1" pin="P$3"/>
-<wire x1="111.76" y1="48.26" x2="91.44" y2="48.26" width="0.1524" layer="91"/>
-<wire x1="91.44" y1="48.26" x2="91.44" y2="43.18" width="0.1524" layer="91"/>
-<pinref part="U$10" gate="G$1" pin="IN"/>
-<label x="93.98" y="48.26" size="1.778" layer="95"/>
+<pinref part="U$1" gate="G$1" pin="P$2"/>
+<wire x1="111.76" y1="45.72" x2="101.6" y2="45.72" width="0.1524" layer="91"/>
+<wire x1="101.6" y1="45.72" x2="101.6" y2="48.26" width="0.1524" layer="91"/>
+<pinref part="U$1" gate="G$1" pin="P$3"/>
+<wire x1="101.6" y1="48.26" x2="111.76" y2="48.26" width="0.1524" layer="91"/>
 </segment>
 </net>
 <net name="N$6" class="0">
 <segment>
-<pinref part="U$9" gate="G$1" pin="P$5"/>
-<wire x1="111.76" y1="63.5" x2="104.14" y2="63.5" width="0.1524" layer="91"/>
-<pinref part="U$9" gate="G$1" pin="P$1"/>
-<wire x1="104.14" y1="63.5" x2="104.14" y2="58.42" width="0.1524" layer="91"/>
-<wire x1="104.14" y1="58.42" x2="111.76" y2="58.42" width="0.1524" layer="91"/>
+<pinref part="D5" gate="G$1" pin="POS"/>
+<wire x1="25.4" y1="60.96" x2="25.4" y2="63.5" width="0.1524" layer="91"/>
+<pinref part="1" gate="G$1" pin="P$2"/>
+<wire x1="60.96" y1="68.58" x2="38.1" y2="68.58" width="0.1524" layer="91"/>
+<wire x1="38.1" y1="68.58" x2="38.1" y2="60.96" width="0.1524" layer="91"/>
+<wire x1="38.1" y1="60.96" x2="25.4" y2="60.96" width="0.1524" layer="91"/>
 </segment>
 </net>
