File: Solar Panel/SolarCellX/SolarCellX_v2_6milmag.brd (EAGLE design)
At the start: 100 x 82 mm, 16 parts

Commit message: Changed pinout for X, added silkscreen
Parts:
- added D6: SB_DIODE, Solar:SB_DIODE
Connections:
- new net N$6: D6.NEG, U$1.P$5
- net N$1: now also U$1.P$2; no longer U$1.P$4
- net V_SOLAR: now also D6.POS; no longer U$1.P$6
Routing:
- net N$6: track 0.00 -> 5.04 mm, vias 0 -> 1
- net N$1: track 54675.6 -> 54677.7 mm
- net V_SOLAR: track 110.3 -> 109.1 mm, vias 1 -> 0
Other:
- board text added: "GND"
- board text added: "MT+"
- board text added: "MT-"
- board text added: "Solar Cell X Board Rev B"
- board text added: "VS"
- board text removed: "PandaSat Solar Cell X Board Rev A"
